File: hw/pcb/led-matrix.kicad_sch (KiCad schematic)
At the start: 130 parts, among them Q1 SSM3K37FSLF, Q10 SSM3K37FSLF, Q2 SSM3K37FSLF, Q3 SSM3K37FSLF, Q4 SSM3K37FSLF, Q5 SSM3K37FSLF, Q6 SSM3K37FSLF, Q7 SSM3K37FSLF, Q8 SSM3K37FSLF, Q9 SSM3K37FSLF

Commit message: fix: added programming and debug port to schematic
Parts:
- D10, D100, D101, D102, D103, D104, D11, D12, D13, D14, D15, D16, D17, D18, D19, D20, D21, D22, D23, D24, D25, D26, D27, D28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: footprint (none) -> Diode_SMD:D_0603_1608Metric
