File: hw/pcb/led-matrix.kicad_sch (KiCad schematic)
At the start: 130 parts, among them Q1 SSM3K37FSLF, Q10 SSM3K37FSLF, Q2 SSM3K37FSLF, Q3 SSM3K37FSLF, Q4 SSM3K37FSLF, Q5 SSM3K37FSLF, Q6 SSM3K37FSLF, Q7 SSM3K37FSLF, Q8 SSM3K37FSLF, Q9 SSM3K37FSLF

Commit message: fix: corrected mosfet footprint
Parts:
- removed Q1, Q10, Q2, Q3, Q4, Q5, Q6, Q7, Q8, Q9: SSM3K37FSLF, Package_TO_SOT_SMD:SOT-416, symbol Transistor_FET:Q_NMOS_DGS
- added Q1, Q10, Q2, Q3, Q4, Q5, Q6, Q7, Q8, Q9: NCH, Package_TO_SOT_SMD:SOT-416, symbol Transistor_FET:Q_NMOS_GSD
Connections:
- net GND: now also Q1.2 (S), Q10.2 (S), Q2.2 (S), Q3.2 (S), Q4.2 (S), Q5.2 (S), Q6.2 (S), Q7.2 (S), Q8.2 (S), Q9.2 (S)
- net at D101.1 (K), D11.1 (K), D21.1 (K)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: now also Q7.3 (D)
- net at D16.1 (K), D26.1 (K), D36.1 (K)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: now also Q2.3 (D)
- net at D17.1 (K), D27.1 (K), D37.1 (K)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: now also Q3.3 (D)
- net at D18.1 (K), D28.1 (K), D38.1 (K)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: now also Q4.3 (D)
- net at R20.2: now also Q5.1 (G)
- net at D102.1 (K), D12.1 (K), D22.1 (K)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: now also Q8.3 (D)
- net at D103.1 (K), D13.1 (K), D23.1 (K)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: now also Q9.3 (D)
- net at D104.1 (K), D14.1 (K), D24.1 (K)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: now also Q10.3 (D)
- net at R25.2: now also Q10.1 (G)
- net at D10.1 (K), D100.1 (K), D20.1 (K)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: now also Q6.3 (D)
- net at R22.2: now also Q7.1 (G)
- net at R21.2: now also Q6.1 (G)
- net at R24.2: now also Q9.1 (G)
- net at D15.1 (K), D25.1 (K), D35.1 (K)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: now also Q1.3 (D)
- net at R16.2: now also Q1.1 (G)
- net at D19.1 (K), D29.1 (K), D39.1 (K)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: now also Q5.3 (D)
- net at R17.2: now also Q2.1 (G)
- net at R18.2: now also Q3.1 (G)
- net at R23.2: now also Q8.1 (G)
- net at R19.2: now also Q4.1 (G)
Other:
- note added: "These LEDs are the APTD1608LSURCK from Kingbright They work with a forward current as low as 2mA (Vf = 1.75V) Hence the large current limiting resistor... (3.3 - Vf) / 0.002 = 775Ω or (3.3 - Vf) / 0.001 = 1550Ω (untested)"
- note removed: "These LEDs are the APTD1608LSURCK from Kingbright They work with a forward current as low as 2mA (Vf = 1.75V) Hence the large current limiting resistor... (3.3 - Vf) / 0.002 = 775Ω"
